File: BO6502 LCD_KEYb/LCD_KEYb_final_rev02.brd (EAGLE design)
At the start: 101.6 x 65 mm, 20 parts, among them IC1 74HCT14N, IC2 74HCT595N, IC3 74HCT595N, IC4 74AC138N, U1 65C22, X1 DIN 5 pin

Commit message: R3 wrong value
Parts:
- R3: value 33K -> 15K
Changed lines of the file:
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@@
 <attribute name="VALUE" x="91.948" y="12.954" size="1.778" layer="27" ratio="10" rot="R90"/>
 </element>
-<element name="R3" library="rcl" library_urn="urn:adsk.eagle:library:334" package="0207/10" package3d_urn="urn:adsk.eagle:package:23491/2" value="33K" x="5.588" y="35.306" smashed="yes" rot="R90">
+<element name="R3" library="rcl" library_urn="urn:adsk.eagle:library:334" package="0207/10" package3d_urn="urn:adsk.eagle:package:23491/2" value="15K" x="5.588" y="35.306" smashed="yes" rot="R90">
 <attribute name="NAME" x="4.064" y="32.258" size="1.27" layer="25" ratio="10" rot="R90"/>
 <attribute name="POPULARITY" value="81" x="5.588" y="35.306" size="1.778" layer="27" rot="R90" display="off"/>
